File: 02_HW/kb_pcb/skeleton/_autosave-skeleton.kicad_pcb (KiCad board)
At the start: 2 copper layers, 65 parts, among them J1 Adafruit_Feather_16_pin, J2 Adafruit_feather_12_pin, SW1 SW_Push, SW10 SW_Push, SW11 SW_Push, SW12 SW_Push, SW13 SW_Push, SW14 SW_Push, SW15 SW_Push, SW16 SW_Push, SW17 SW_Push, SW18 SW_Push, SW19 SW_Push, SW2 SW_Push, SW20 SW_Push, SW21 SW_Push, SW22 SW_Push, SW23 SW_Push, SW24 SW_Push, SW25 SW_Push, SW26 SW_Push, SW27 SW_Push, SW28 SW_Push, SW29 SW_Push, SW3 SW_Push, SW30 SW_Push, SW4 SW_Push, SW6 SW_Push, SW7 SW_Push, SW8 SW_Push, SW9 SW_Push

Commit message: moved thumb pad, fixed net labels,added design rules
Parts:
- moved R1 9.51 mm to (169.7, 106.0)
- moved R2 9.51 mm to (169.7, 108.5)
- moved R3 9.51 mm to (169.7, 111.0)
- moved R4 9.51 mm to (169.7, 113.5)
- moved R5 9.51 mm to (169.7, 116.0)
- moved D1 7.66 mm to (155.1, 166.0)
- moved D11 7.66 mm to (155.1, 127.9)
- moved D16 7.66 mm to (136.0, 147.0)
- moved D21 7.66 mm to (136.0, 127.9)
- moved D26 7.66 mm to (117.0, 127.9)
- moved D6 7.66 mm to (155.1, 147.0)
- moved SW1 7.66 mm to (157.6, 170.5)
- moved SW11 7.66 mm to (157.6, 132.4)
- moved SW16 7.66 mm to (138.5, 151.4)
- moved SW21 7.66 mm to (138.5, 132.4)
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Connections:
- J1 pad 10: unconnected-(J1-Pin_10-Pad10) -> /Col_4
- J1 pad 11: unconnected-(J1-Pin_11-Pad11) -> /Col_5
- J1 pad 6: unconnected-(J1-Pin_6-Pad6) -> /Col_0
- J1 pad 7: unconnected-(J1-Pin_7-Pad7) -> /Col_1
- J1 pad 8: unconnected-(J1-Pin_8-Pad8) -> /Col_2
- J1 pad 9: unconnected-(J1-Pin_9-Pad9) -> /Col_3
- J2 pad 1: /Col_0 -> unconnected-(J2-Pin_1-Pad1)
- J2 pad 10: /Row_3 -> /Row_2
- J2 pad 11: /Row_4 -> /Row_1
- J2 pad 12: unconnected-(J2-Pin_12-Pad12) -> /Row_0
- J2 pad 2: /Col_1 -> unconnected-(J2-Pin_2-Pad2)
- J2 pad 3: /Col_2 -> unconnected-(J2-Pin_3-Pad3)
- J2 pad 4: /Col_3 -> unconnected-(J2-Pin_4-Pad4)
- J2 pad 5: /Col_4 -> unconnected-(J2-Pin_5-Pad5)
- J2 pad 6: /Col_5 -> unconnected-(J2-Pin_6-Pad6)
- J2 pad 7: /Row_0 -> unconnected-(J2-Pin_7-Pad7)
- J2 pad 8: /Row_1 -> /Row_4
- J2 pad 9: /Row_2 -> /Row_3
Other:
- rule pad_to_mask_clearance: 0 -> 0.038
