File: 02_HW/kb_pcb/keybird/keybird.kicad_sch (KiCad schematic)
At the start: 65 parts, among them J1 Adafruit_Feather_16_pin, J2 Adafruit_feather_12_pin, SW1 SW_Push, SW10 SW_Push, SW11 SW_Push, SW12 SW_Push, SW13 SW_Push, SW14 SW_Push, SW15 SW_Push, SW16 SW_Push, SW17 SW_Push, SW18 SW_Push, SW19 SW_Push, SW2 SW_Push, SW20 SW_Push, SW21 SW_Push, SW22 SW_Push, SW23 SW_Push, SW24 SW_Push, SW25 SW_Push, SW26 SW_Push, SW27 SW_Push, SW28 SW_Push, SW29 SW_Push, SW3 SW_Push, SW30 SW_Push, SW4 SW_Push, SW6 SW_Push, SW7 SW_Push, SW8 SW_Push, SW9 SW_Push

Commit message: Reverseddiodes for active low implementation
Connections:
- net Row_0: now also D1.2 (A), D11.2 (A), D16.2 (A), D21.2 (A), D26.2 (A), D6.2 (A); no longer D1.1 (K), D11.1 (K), D16.1 (K), D21.1 (K), D26.1 (K), D6.1 (K)
- net Row_1: now also D12.2 (A), D17.2 (A), D2.2 (A), D22.2 (A), D27.2 (A), D7.2 (A); no longer D12.1 (K), D17.1 (K), D2.1 (K), D22.1 (K), D27.1 (K), D7.1 (K)
- net Row_2: now also D13.2 (A), D18.2 (A), D23.2 (A), D28.2 (A), D3.2 (A), D8.2 (A); no longer D13.1 (K), D18.1 (K), D23.1 (K), D28.1 (K), D3.1 (K), D8.1 (K)
- net Row_3: now also D14.2 (A), D19.2 (A), D24.2 (A), D29.2 (A), D4.2 (A), D9.2 (A); no longer D14.1 (K), D19.1 (K), D24.1 (K), D29.1 (K), D4.1 (K), D9.1 (K)
- net Row_4: now also D10.2 (A), D15.2 (A), D20.2 (A), D25.2 (A), D30.2 (A); no longer D10.1 (K), D15.1 (K), D20.1 (K), D25.1 (K), D30.1 (K)
- net at SW29.2: now also D29.1 (K); no longer D29.2 (A)
- net at SW2.2: now also D2.1 (K); no longer D2.2 (A)
- net at SW22.2: now also D22.1 (K); no longer D22.2 (A)
- net at SW8.2: now also D8.1 (K); no longer D8.2 (A)
- net at SW16.2: now also D16.1 (K); no longer D16.2 (A)
- net at SW3.2: now also D3.1 (K); no longer D3.2 (A)
- net at SW10.2: now also D10.1 (K); no longer D10.2 (A)
- net at SW28.2: now also D28.1 (K); no longer D28.2 (A)
- net at SW25.2: now also D25.1 (K); no longer D25.2 (A)
- net at SW27.2: now also D27.1 (K); no longer D27.2 (A)
- net at SW20.2: now also D20.1 (K); no longer D20.2 (A)
- net at SW4.2: now also D4.1 (K); no longer D4.2 (A)
- net at SW18.2: now also D18.1 (K); no longer D18.2 (A)
- net at SW24.2: now also D24.1 (K); no longer D24.2 (A)
- net at SW6.2: now also D6.1 (K); no longer D6.2 (A)
- net at SW21.2: now also D21.1 (K); no longer D21.2 (A)
- net at SW15.2: now also D15.1 (K); no longer D15.2 (A)
- net at SW23.2: now also D23.1 (K); no longer D23.2 (A)
- net at SW30.2: now also D30.1 (K); no longer D30.2 (A)
- net at SW9.2: now also D9.1 (K); no longer D9.2 (A)
- net at SW1.2: now also D1.1 (K); no longer D1.2 (A)
- net at SW19.2: now also D19.1 (K); no longer D19.2 (A)
- net at SW26.2: now also D26.1 (K); no longer D26.2 (A)
- net at SW13.2: now also D13.1 (K); no longer D13.2 (A)
- net at SW7.2: now also D7.1 (K); no longer D7.2 (A)
- net at SW17.2: now also D17.1 (K); no longer D17.2 (A)
- net at SW12.2: now also D12.1 (K); no longer D12.2 (A)
- net at SW14.2: now also D14.1 (K); no longer D14.2 (A)
- net at SW11.2: now also D11.1 (K); no longer D11.2 (A)
Other:
- moved on the sheet: D1, D10, D11, D12, D13, D14, D15, D16, D17, D18, D19, D2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
