File: 02_HW/kb_pcb/keybird_left/keybird_left.kicad_pcb (KiCad board)
At the start: 2 copper layers, 152.4 x 148.3 mm, 79 parts, among them J1 Adafruit_Feather_16_pin, J2 Adafruit_feather_12_pin, J4 FTDI UART, SW1 SW_Push, SW10 SW_Push, SW11 SW_Push, SW12 SW_Push, SW13 SW_Push, SW14 SW_Push, SW15 SW_Push, SW16 SW_Push, SW17 SW_Push, SW18 SW_Push, SW19 SW_Push, SW2 SW_Push, SW20 SW_Push, SW21 SW_Push, SW22 SW_Push, SW23 SW_Push, SW24 SW_Push, SW25 SW_Push, SW26 SW_Push, SW27 SW_Push, SW28 SW_Push, SW29 SW_Push, SW3 SW_Push, SW30 SW_Push, SW4 SW_Push, SW5 Power enable, SW6 SW_Push, SW7 SW_Push, SW8 SW_Push, SW9 SW_Push

Commit message: left and right board pass design rule checks
Parts:
- moved H4 26.5 mm to (116.0, 101.0)
- moved D22 2.00 mm to (109.4, 101.0)
Routing:
- net /Row_1: track 130.6 -> 132.4 mm
- net Net-(D22-K): track 5.37 -> 6.20 mm
- net GNDREF: vias 229 -> 226

Commit message: Left and right boards pass design rule checks
Parts:
- J1: footprint Connector_PinHeader_2.54mm:PinHeader_1x16_P2.54mm_Vertical -> Connector_PinSocket_2.54mm:PinSocket_1x16_P2.54mm_Vertical
- J2: footprint Connector_PinHeader_2.54mm:PinHeader_1x12_P2.54mm_Vertical -> Connector_PinSocket_2.54mm:PinSocket_1x12_P2.54mm_Vertical
Routing:
- net /RED_LED: track 21.5 -> 22.1 mm
- net GNDREF: vias 226 -> 228
Changed lines of the file:
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@@
 		)
 	)
-	(footprint "Connector_PinHeader_2.54mm:PinHeader_1x16_P2.54mm_Vertical"
+	(footprint "Connector_PinSocket_2.54mm:PinSocket_1x16_P2.54mm_Vertical"
 		(locked yes)
 		(layer "F.Cu")
 		(at 140.705 75.375)
-		(descr "Through hole straight pin header, 1x16, 2.54mm pitch, single row")
-		(tags "Through hole pin header THT 1x16 2.54mm single row")
+		(descr "Through hole straight socket strip, 1x16, 2.54mm pitch, single row (from Kicad 4.0.7), script generated")
+		(tags "Through hole socket strip THT 1x16 2.54mm single row")
 		(property "Reference" "J1"
-			(at 0 -2.33 0)
+			(at 0 -2.77 0)
 			(layer "F.SilkS")
 			(effects
@@
 		)
 		(property "Value" "Adafruit_Feather_16_pin"
-			(at 0 40.43 0)
+			(at 0 40.87 0)
 			(layer "F.Fab")
-			(hide yes)
 			(effects
 				(font
@@
 			)
 		)
-		(property "Footprint" "Connector_PinHeader_2.54mm:PinHeader_1x16_P2.54mm_Vertical"
+		(property "Footprint" "Connector_PinSocket_2.54mm:PinSocket_1x16_P2.54mm_Vertical"
 			(at 0 0 0)
 			(unlocked yes)
@@
 		(attr through_hole)
 		(fp_line
-			(start -1.33 -1.33)
-			(end 0 -1.33)
+			(start -1.33 1.27)
+			(end -1.33 39.43)
 			(stroke
 				(width 0.12)
@@
 		)
 		(fp_line
-			(start -1.33 0)
-			(end -1.33 -1.33)
+			(start -1.33 1.27)
+			(end 1.33 1.27)
 			(stroke
 				(width 0.12)
@@
 		)
 		(fp_line
-			(start -1.33 1.27)
-			(end -1.33 39.43)
+			(start -1.33 39.43)
+			(end 1.33 39.43)
 			(stroke
 				(width 0.12)
@@
 		)
 		(fp_line
-			(start -1.33 1.27)
-			(end 1.33 1.27)
+			(start 0 -1.33)
+			(end 1.33 -1.33)
 			(stroke
 				(width 0.12)
@@
 		)
 		(fp_line
-			(start -1.33 39.43)
-			(end 1.33 39.43)
+			(start 1.33 -1.33)
+			(end 1.33 0)
 			(stroke
 				(width 0.12)
@@
 		(fp_line
 			(start -1.8 -1.8)
-			(end -1.8 39.9)
+			(end 1.75 -1.8)
 			(stroke
 				(width 0.05)
@@
 		(fp_line
 			(start -1.8 39.9)
-			(end 1.8 39.9)
+			(end -1.8 -1.8)
 			(stroke
 				(width 0.05)
@@
 		)
 		(fp_line
-			(start 1.8 -1.8)
-			(end -1.8 -1.8)
+			(start 1.75 -1.8)
+			(end 1.75 39.9)
 			(stroke
 				(width 0.05)
@@
 		)
 		(fp_line
-			(start 1.8 39.9)
-			(end 1.8 -1.8)
+			(start 1.75 39.9)
+			(end -1.8 39.9)
 			(stroke
 				(width 0.05)
@@
 		)
 		(fp_line
-			(start -1.27 -0.635)
-			(end -0.635 -1.27)
+			(start -1.27 -1.27)
+			(end 0.635 -1.27)
 			(stroke
 				(width 0.1)
@@
 		(fp_line
 			(start -1.27 39.37)
-			(end -1.27 -0.635)
+			(end -1.27 -1.27)
 			(stroke
 				(width 0.1)
@@
 		)
 		(fp_line
-			(start -0.635 -1.27)
-			(end 1.27 -1.27)
+			(start 0.635 -1.27)
+			(end 1.27 -0.635)
 			(stroke
 				(width 0.1)
@@
 		)
 		(fp_line
-			(start 1.27 -1.27)
+			(start 1.27 -0.635)
 			(end 1.27 39.37)
 			(stroke
@@
 			(pintype "passive")
 		)
-		(model "${KICAD8_3DMODEL_DIR}/Connector_PinHeader_2.54mm.3dshapes/PinHeader_1x16_P2.54mm_Vertical.wrl"
+		(model "${KICAD8_3DMODEL_DIR}/Connector_PinSocket_2.54mm.3dshapes/PinSocket_1x16_P2.54mm_Vertical.wrl"
 			(offset
 				(xyz 0 0 0)
@@
 		)
 	)
-	(footprint "Connector_PinHeader_2.54mm:PinHeader_1x12_P2.54mm_Vertical"
+	(footprint "Connector_PinSocket_2.54mm:PinSocket_1x12_P2.54mm_Vertical"
 		(locked yes)
 		(layer "F.Cu")
 		(at 161 85.525)
-		(descr "Through hole straight pin header, 1x12, 2.54mm pitch, single row")
-		(tags "Through hole pin header THT 1x12 2.54mm single row")
+		(descr "Through hole straight socket strip, 1x12, 2.54mm pitch, single row (from Kicad 4.0.7), script generated")
+		(tags "Through hole socket strip THT 1x12 2.54mm single row")
 		(property "Reference" "J2"
-			(at 0 -2.33 0)
+			(at 0 -2.77 0)
 			(layer "F.SilkS")
 			(effects
@@
 		)
 		(property "Value" "Adafruit_feather_12_pin"
-			(at 0 30.27 0)
+			(at 0 30.71 0)
 			(layer "F.Fab")
-			(hide yes)
 			(effects
 				(font
@@
 			)
 		)
-		(property "Footprint" "Connector_PinHeader_2.54mm:PinHeader_1x12_P2.54mm_Vertical"
+		(property "Footprint" "Connector_PinSocket_2.54mm:PinSocket_1x12_P2.54mm_Vertical"
 			(at 0 0 0)
 			(unlocked yes)
@@
 		(attr through_hole)
 		(fp_line
-			(start -1.33 -1.33)
-			(end 0 -1.33)
+			(start -1.33 1.27)
+			(end -1.33 29.27)
 			(stroke
 				(width 0.12)
@@
 		)
 		(fp_line
-			(start -1.33 0)
-			(end -1.33 -1.33)
+			(start -1.33 1.27)
+			(end 1.33 1.27)
 			(stroke
 				(width 0.12)
@@
 		)
 		(fp_line
-			(start -1.33 1.27)
-			(end -1.33 29.27)
+			(start -1.33 29.27)
+			(end 1.33 29.27)
 			(stroke
 				(width 0.12)
@@
 		)
 		(fp_line
-			(start -1.33 1.27)
-			(end 1.33 1.27)
+			(start 0 -1.33)
+			(end 1.33 -1.33)
 			(stroke
 				(width 0.12)
@@
 		)
 		(fp_line
-			(start -1.33 29.27)
-			(end 1.33 29.27)
+			(start 1.33 -1.33)
+			(end 1.33 0)
 			(stroke
 				(width 0.12)
@@
 		(fp_line
 			(start -1.8 -1.8)
-			(end -1.8 29.75)
+			(end 1.75 -1.8)
 			(stroke
 				(width 0.05)
@@
 		)
 		(fp_line
-			(start -1.8 29.75)
-			(end 1.8 29.75)
+			(start -1.8 29.7)
+			(end -1.8 -1.8)
 			(stroke
 				(width 0.05)
@@
 		)
 		(fp_line
-			(start 1.8 -1.8)
-			(end -1.8 -1.8)
+			(start 1.75 -1.8)
+			(end 1.75 29.7)
 			(stroke
 				(width 0.05)
@@
 		)
 		(fp_line
-			(start 1.8 29.75)
-			(end 1.8 -1.8)
+			(start 1.75 29.7)
+			(end -1.8 29.7)
 			(stroke
 				(width 0.05)
@@
 		)
 		(fp_line
-			(start -1.27 -0.635)
-			(end -0.635 -1.27)
+			(start -1.27 -1.27)
+			(end 0.635 -1.27)
 			(stroke
 				(width 0.1)
@@
 		(fp_line
 			(start -1.27 29.21)
-			(end -1.27 -0.635)
+			(end -1.27 -1.27)
 			(stroke
 				(width 0.1)
@@
 		)
 		(fp_line
-			(start -0.635 -1.27)
-			(end 1.27 -1.27)
+			(start 0.635 -1.27)
+			(end 1.27 -0.635)
 			(stroke
 				(width 0.1)
@@
 		)
 		(fp_line
-			(start 1.27 -1.27)
+			(start 1.27 -0.635)
 			(end 1.27 29.21)
 			(stroke
@@
 			(pintype "passive")
 		)
-		(model "${KICAD8_3DMODEL_DIR}/Connector_PinHeader_2.54mm.3dshapes/PinHeader_1x12_P2.54mm_Vertical.wrl"
+		(model "${KICAD8_3DMODEL_DIR}/Connector_PinSocket_2.54mm.3dshapes/PinSocket_1x12_P2.54mm_Vertical.wrl"
 			(offset
 				(xyz 0 0 0)
@@
 	)
 	(via
+		(at 134.965599 120.592633)
+		(size 1)
+		(drill 0.5)
+		(layers "F.Cu" "B.Cu")
+		(free yes)
+		(net 43)
+	)
+	(via
 		(at 29 108)
 		(size 1)
@@
 	)
 	(via
+		(at 147.041801 121.722737)
+		(size 1)
+		(drill 0.5)
+		(layers "F.Cu" "B.Cu")
+		(free yes)
+		(net 43)
+	)
+	(via
 		(at 104 48)
 		(size 1)
@@
 	)
 	(segment
-		(start 138 71.732202)
+		(start 137.767346 71.964856)
 		(end 141.67 68.062202)
 		(width 0.3)
@@
 	)
 	(segment
-		(start 140.705 85.535)
-		(end 138 82.83)
+		(start 137.767346 83.217146)
+		(end 137.767346 71.964856)
 		(width 0.3)
 		(layer "F.Cu")
@@
 	)
 	(segment
-		(start 138 82.83)
-		(end 138 71.732202)
+		(start 140.0852 85.535)
+		(end 137.767346 83.217146)
 		(width 0.3)
 		(layer "F.Cu")
@@
 	)
 	(segment
-		(start 137.5 63.155693)
-		(end 141.63 59.025693)
+		(start 140.705 85.535)
+		(end 140.0852 85.535)
+		(width 0.3)
+		(layer "F.Cu")
+		(net 48)
+	)
+	(segment
+		(start 140.705 88.075)
+		(end 137.077132 84.447132)
 		(width 0.3)
 		(layer "F.Cu")
@@
 	)
 	(segment
-		(start 141.63 59.025693)
-		(end 141.63 57.7)
+		(start 137.077132 63.578561)
+		(end 141.63 59.025693)
 		(width 0.3)
 		(layer "F.Cu")
@@
 	)
 	(segment
-		(start 137.5 84.87)
-		(end 137.5 63.155693)
+		(start 137.077132 84.447132)
+		(end 137.077132 63.578561)
 		(width 0.3)
 		(layer "F.Cu")
@@
 	)
 	(segment
-		(start 140.705 88.075)
-		(end 137.5 84.87)
+		(start 141.63 59.025693)
+		(end 141.63 57.7)
 		(width 0.3)
 		(layer "F.Cu")
@@
 	)
 	(segment
-		(start 141.65 50.741628)
-		(end 141.65 48.732)
+		(start 140.705 90.615)
+		(end 136.231939 86.141939)
 		(width 0.3)
 		(layer "F.Cu")
@@
 	)
 	(segment
-		(start 136.5 55.891628)
+		(start 136.231939 56.159689)
 		(end 141.65 50.741628)
 		(width 0.3)
@@
 	)
 	(segment
-		(start 136.5 86.41)
-		(end 136.5 55.891628)
+		(start 141.65 50.741628)
+		(end 141.65 48.732)
 		(width 0.3)
 		(layer "F.Cu")
@@
 	)
 	(segment
-		(start 140.705 90.615)
-		(end 136.5 86.41)
+		(start 136.231939 86.141939)
+		(end 136.231939 56.159689)
 		(width 0.3)
 		(layer "F.Cu")
@@
 			(clearance 0.5)
 		)
-		(min_thickness 0.25)
+		(min_thickness 0.5)
 		(filled_areas_thickness no)
 		(fill yes
